File: AttenuatorX/Digital Attenuator.sch (KiCad schematic (older format))
At the start: 27 parts

Commit message: Updated Schematics
Parts:
- removed C? (x6): 100pF, symbol C
- removed U?: SKY13268-344, symbol SKY13268-344
- removed U?: LT5538IDD, symbol LT5538IDD
- added A1, A2, A? (x2): 3, symbol R
- added A? (x2): 10, symbol R
- added C? (x3): 47pF, symbol C
- added C? (x4): 1nF, symbol C
- added C?: 0.1uF, symbol C
- added C? (x6): 330pF, symbol C
- added C? (x3): 0.2pF, symbol C
- added C?: 10pF, symbol C
- added R? (x4): 33, symbol R
- added R? (x2): 2.5k, symbol R
- added R? (x2): 1M, symbol R
- added U?: LT5534, symbol LT5534
- added X? (x3): RF_CONN, symbol RF_CONN
Connections:
- net GND: now also U?.14 (GND), U?.17 (PUP2), U?.18 (PUP1), U?.5 (GND), U?.PDL (GND), C?.1, C?.1, C?.1, C?.1, C?.1, C?.1, C?.1, C?.1, C?.1, C?.1, C?.2, C?.2, C?.2, C?.2, C?.2, C?.2, U?.2 (GND), U?.5 (GND), X?.2, X?.2, X?.2
- net at U?.5 (J1): now also C?.1
- net at U?.11 (ANT_RF): now also C?.1
- net at U?.13 (RF1): now also A?.2
- net at U?.15 (RF2): now also C?.1
- net at U?.2 (VDD): now also R?.2, R?.2
- net at U?.3 (V2): now also C?.1, R?.1
- net at U?.4 (V1): now also C?.1, R?.1
- net at U?.6 (RF4): now also C?.1
- net at U?.8 (RF3): now also C?.1
- net at U?.14 (ATT_OUT): now also C?.1
- net at U?.10 (ACGND4): now also C?.2
- net at U?.11 (ACGND5): now also C?.2; no longer U?.12 (ACGND6)
- net at U?.13 (RF_OUT): now also C?.2
- net at U?.18 (VDD): now also C?.1, R?.2
- net at U?.2 (CLK): now also C?.2, R?.2
- net at U?.3 (SERIN): now also C?.2, R?.2
- net at U?.4 (LE): now also C?.2, R?.2
- net at U?.6 (RF_IN): now also C?.2
- net at U?.7 (ACGND1), U?.8 (ACGND2): now also U?.9 (ACGND3), C?.2
- net at C?.1: now also A?.1 (x2)
- net at C?.1: now also A2.1
- net at C?.1: now also U?.6 (RF)
- new net: C?.2, U?.12 (ACGND6)
- new net: R?.1, U?.1 (EN)
- new net: R?.2, U?.3 (VOUT)
- new net: C?.1, C?.2, X?.1 (RF)
- new net: A1.1, A2.2
- new net: A1.2, C?.2, X?.1 (RF)
- new net: A?.2, C?.2, X?.1 (RF)
- new net: A?.1, A?.2 (x2)
- new net 5V: C?.1, C?.1, R?.1, R?.2, U?.4 (VCC)
- new net CLK: R?.1
- new net LE: R?.1
- new net SERIN: R?.1
- new net VOUT: C?.1, R?.1
- no-connect marks 0 -> 1
Other:
- moved on the sheet: C?, U?
