File: AttenuatorXLE/AttenuatorXLE.sch (KiCad schematic (older format))
At the start: 20 parts

Commit message: Updated Schematics
Parts:
- removed C?: C, symbol C
- removed X?: RF_CONN, symbol RF_CONN
- added A1: 2, symbol R
- added A2, A3: 3, symbol R
- added A4, A5: 20, symbol R
- added C1, C8: 0.1uF, symbol C
- added C15: 10pF, symbol C
- added C2: 4.7uF, symbol C
- added C20, C6: 0.2pF, symbol C
- added C3, C4, C9: 100pF, symbol C
- added P1: CONN_8, symbol CONN_8
- added R1, R3: 2.5k, symbol R
- added R2: 33, symbol R
- added U3: LT5534, symbol LT5534
- added X2: RF_CONN, symbol RF_CONN
- C10, C11, C13, C14: renamed from C?; value C -> 330pF
- C12: renamed from C?; value C -> 0.1uF
- C16, C18: renamed from C?; value C -> 1nF
- C17, C19, C21: renamed from C?; value C -> 47pF
- C5, C7: renamed from C?; value C -> 100pF
- R4, R5, R6: renamed from R?; value R -> 33
- gave numbers to parts that had none: 3
Connections:
- net GND: now also C1.1, C15.2, C2.1, C20.1, C3.1, C4.1, C6.1, C8.1, C9.1, P1.2 (P2), U3.2 (GND), U3.5 (GND), X2.2
- net at U1.1 (J2): now also C16.1; no longer C5.2
- net at U1.3 (J3): now also A4.1; no longer C7.2
- net V2: now reaches U1.4 (V2)
- net V2: now also C4.2, P1.7 (P7)
- net at U1.5 (J1): now also C5.2
- net V1: now reaches U1.6 (V1)
- net V1: now also C3.2, P1.6 (P6)
- net at C5.1: now also A3.2
- net at C7.1: now also U3.6 (RF); no longer X1.1 (RF)
- net at C18.1: now also C20.2, X2.1 (RF)
- net LE: now reaches R4.1
- net LE: now also P1.5 (P5)
- net CLK: now reaches R5.1
- net CLK: now also P1.4 (P4)
- net SERIN: now reaches R6.1
- net SERIN: now also P1.3 (P3)
- net +5V: no longer names the net of C12.1, U2.18 (VDD)
- net +5V: now also R2.2
- new net: A5.2, C7.2
- new net: A1.1, C6.2, X1.1 (RF)
- new net: A2.2, A3.1
- new net: A1.2, A2.1
- new net: R1.2, U3.1 (EN)
- new net: R3.2, U3.3 (VOUT)
- new net: A4.2, A5.1
- new net 5V: C1.2, C2.2, C8.2, C9.2, P1.1 (P1), R1.1, R2.1, U3.4 (VCC)
- new net VOUT: C15.1, P1.8 (P8), R3.1
- no-connect marks 0 -> 1
Other:
- note added: "Input\nDecoupling"
- moved on the sheet: C10, C11, C12, C13, C14, C16, C17, C18, C19, C21, C5, C7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

Commit message: Updated BOM and Libraries
Connections:
- net V1: now also P1.7 (P7); no longer P1.6 (P6)
- net V2: now also P1.8 (P8); no longer P1.7 (P7)
- net VOUT: now also P1.6 (P6); no longer P1.8 (P8)
Changed lines of the file:
@@
-EESchema Schematic File Version 2  date 11/26/2011 4:25:13 PM
+EESchema Schematic File Version 2  date 11/30/2011 4:16:59 PM
 LIBS:power
 LIBS:device
@@
 LIBS:contrib
 LIBS:valves
-LIBS:AttenuatorX
 LIBS:AttenuatorXLE-cache
 EELAYER 25  0
@@
 Sheet 1 1
 Title "AttenuatorXLE"
-Date "26 nov 2011"
+Date "30 nov 2011"
 Rev "1"
 Comp "Projects and Stuff LLC"
@@
 Comment4 "Control Voltage: +5V"
 $EndDescr
+Text Label 2700 5400 2    60   ~ 0
+V1
 NoConn ~ 7950 3050
 Wire Wire Line
@@
 	2800 4900 2700 4900
 Wire Wire Line
-	2800 5400 2700 5400
+	2800 5500 2700 5500
 Wire Wire Line
 	2800 5200 2700 5200
@@
 	2800 5100 2700 5100
 Wire Wire Line
+	2800 5400 2700 5400
+Wire Wire Line
 	2800 5300 2700 5300
-Wire Wire Line
-	2800 5500 2700 5500
 Wire Wire Line
 	2800 4800 2700 4800
@@
 Text Label 2700 5200 2    60   ~ 0
 LE
+Text Label 2700 5300 2    60   ~ 0
+VOUT
 Text Label 2700 5500 2    60   ~ 0
-VOUT
-Text Label 2700 5400 2    60   ~ 0
 V2
-Text Label 2700 5300 2    60   ~ 0
-V1
 $Comp
 L GND #PWR04
